File: pcbs/right_thumbs_rev1.2.kicad_pcb (KiCad board)
At the start: 2 copper layers, 93.5 x 38.7 mm, 12 parts

Commit message: Revision 1.2 - Socket was moved from middle home to inner home - Vertical column connections became thinner
Connections:
- BAT1 pad 2: RBATN -> RGND
Routing:
- net RGND: track 12.6 -> 49.5 mm
- net RBATN: track 23.8 -> 0.00 mm
- net CT10: track 15.4 -> 11.6 mm
- net CT7: track 65.1 -> 67.0 mm
- net CT8: track 43.5 -> 41.8 mm, vias 1 -> 3
- net RBATP: track 16.6 -> 17.7 mm
- net CT6: track 88.7 -> 89.7 mm, vias 2 -> 0
- net CT9: track 11.7 -> 11.1 mm, vias 0 -> 1
Other:
- board text added: "NKB rev1.2 right"
