File: pcbs/right_rev1.2_2mm.kicad_pcb (KiCad board)
At the start: 2 copper layers, 101 x 79 mm, 31 parts

Commit message: revision 1.3 - 2mm column connections - minimized switch area
Other:
- board text added: "LIKEeb"
- board text added: "right"
Changed lines of the file:
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@@
   (gr_line (start 236.291967 66.91441) (end 243.291967 66.91441)
     (stroke (width 0.15) (type solid)) (layer "Edge.Cuts"))
+  (gr_text "right" (at 233.48 86.84) (layer "Edge.Cuts")
+    (effects (font (size 1 1) (thickness 0.15)) (justify left bottom))
+  )
+  (gr_text "LIKEeb" (at 231.51 85.38) (layer "Edge.Cuts")
+    (effects (font (size 1.5 1.5) (thickness 0.15) italic) (justify left bottom))
+  )
   (segment (start 238.27059 84.80941) (end 242.27059 80.80941) (width 0.25) (layer "F.Cu") (net 1))
   (segment (start 255.841396 90.405) (end 256.320305 90.405) (width 0.25) (layer "F.Cu") (net 1))
